File: ehx-hazarai-mod.kicad_pcb (KiCad board)
At the start: 2 copper layers, 35.8 x 34.3 mm, 31 parts, among them P1 in filt, P2 fsw +, P3 loop in, P4 beat in, P5 beat out, P6 loop out, P7 5v in, P8 in nofilt, P9 fsw gnd, Q1 BC547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

Commit message: updated connections and i/o.. should work now..
needs a little more layout
Parts:
- removed R10: 1k, Resistors_ThroughHole:Resistor_Vertical_RM5mm
- added P10: inv loop out, Pin_Headers:Pin_Header_Straight_1x01_Pitch2.54mm, F.Cu at (146.5, 124.5)
- P1, P2, P3, P4, P5, P6, P7, P8, P9: footprint Pin_Headers:Pin_Header_Straight_1x01 -> Pin_Headers:Pin_Header_Straight_1x01_Pitch2.54mm
- R12: value 10k -> 3k3
- R15: value 620R -> 3k3
- R9: value 620R -> 33k
- moved Q4 1.32 mm to (145.9, 134.4), turned to 180 degrees
Connections:
- Q2 pad 1: Net-(Q2-Pad1) -> Net-(P10-Pad1)
- Q4 pad 1: Net-(Q4-Pad1) -> Net-(P6-Pad1)
- R12 pad 2: Net-(R10-Pad1) -> Net-(P10-Pad1)
- R15 pad 1: Net-(Q4-Pad1) -> Net-(P6-Pad1)
- R15 pad 2: Net-(P6-Pad1) -> GND
- R9 pad 2: Net-(R10-Pad1) -> Net-(P10-Pad1)
Routing:
- net Net-(P10-Pad1): track 0.00 -> 27.9 mm
- net GND: track 36.5 -> 59.7 mm
- net Net-(R10-Pad1): track 18.2 -> 0.00 mm
- net +5V: track 42.9 -> 36.5 mm
- net Net-(Q4-Pad1): track 4.08 -> 0.00 mm
- net Net-(Q2-Pad1): track 2.90 -> 0.00 mm
- net Net-(P6-Pad1): track 7.58 -> 10.3 mm
Other:
- board text added: "xnor 4/17"
- board text removed: "xnor 10/16"
